File: MAX30102_rigid.kicad_pcb (KiCad board)
At the start: 2 copper layers, 7 parts, among them U1 MAX30102

Commit message: Update for Ver2.0
Parts:
- added C1: 4.7μ, MyLibrary:C0603, B.Cu at (119.2, 92.0)
- added C2: 4.7μ, MyLibrary:C0603, F.Cu at (126.0, 86.1)
- added C3: 4.7μ, MyLibrary:C0603, B.Cu at (116.5, 86.1)
- added C4: 0.1μ, Capacitor_SMD:C_0402_1005Metric, F.Cu at (122.0, 86.5)
- added C5: 10μ, MyLibrary:C0603, F.Cu at (116.7, 88.0)
- added C6: 0.1μ, Capacitor_SMD:C_0402_1005Metric, F.Cu at (119.0, 86.3)
- added C7: 0.1μ, Capacitor_SMD:C_0402_1005Metric, B.Cu at (127.1, 92.4)
- added C8: 0.1μ, Capacitor_SMD:C_0402_1005Metric, F.Cu at (121.2, 92.7)
- added FPC1: ~, MyLibrary:FPC-SMD_AFC07-S05FCC-00, B.Cu at (122.5, 88.5)
- added U2: ~, MyLibrary:SOT-23-5_L2.9-W1.6-P0.95-LS2.8-BL, B.Cu at (116.5, 91.7)
- added U3: ~, MyLibrary:MICROPARK_L1.6-W1.6-P0.50-BL-1, B.Cu at (123.0, 92.3)
- R1, R2, R3: footprint Resistor_SMD:R_0603_1608Metric -> Resistor_SMD:R_0402_1005Metric
- R4, R5, R6: footprint Resistor_SMD:R_0603_1608Metric -> Resistor_SMD:R_0402_1005Metric; moved to B.Cu
- moved R1 152.7 mm to (123.8, 92.3), turned to -90 degrees
- moved R4 150.0 mm to (126.7, 90.9)
- moved R2 148.4 mm to (120.2, 92.2), turned to 90 degrees
- moved R5 147.5 mm to (127.2, 87.8), turned to 90 degrees
- moved R6 147.3 mm to (127.5, 89.7), turned to 180 degrees
- moved U1 144.4 mm to (121.9, 89.3), turned to 90 degrees
- moved R3 143.5 mm to (120.4, 86.2), turned to -90 degrees
Routing:
- net +3.3V: track 0.00 -> 37.0 mm, vias 0 -> 4
- net GND: track 0.00 -> 29.2 mm, vias 0 -> 6
- net Net-(U1-VDD): track 0.00 -> 21.9 mm, vias 0 -> 2
- net Net-(U3-A0): track 0.00 -> 12.7 mm
- net Net-(U1-SDA): track 0.00 -> 9.94 mm, vias 0 -> 1
- net Net-(U3-A1): track 0.00 -> 6.88 mm
- net Net-(U1-SCL): track 0.00 -> 5.25 mm, vias 0 -> 1
- net Net-(U3-OE): track 0.00 -> 4.11 mm
- net Net-(U1-~{INT}): track 0.00 -> 4.09 mm, vias 0 -> 1
- added copper zone on B.Cu, net GND
- added copper zone on F.Cu, net GND
Other:
- board outline added: 15 x 10 mm
- board text added: "I.TAKATO"
- board text added: "MAX2.0"
