File: MAX30102_rigid.kicad_sch (KiCad schematic)
At the start: 18 parts, among them U1 MAX30102

Commit message: Update for Ver2.0
Parts:
- C4, C6, C7, C8: footprint MyLibrary:C0603 -> Capacitor_SMD:C_0402_1005Metric
- FPC1, U2, U3: value ~ -> (none)
- R1, R2, R3, R4, R5, R6: footprint Resistor_SMD:R_0603_1608Metric -> Resistor_SMD:R_0402_1005Metric
